File: PCB/Haptics PWM module/Haptics PWM module.kicad_pcb (KiCad board)
At the start: 2 copper layers, 47 x 34.5 mm, 23 parts, among them J1 Conn_01x05_Pin, J2 JST_XH_FEMALE, J3 JST_XH_FEMALE_1, U1 ULN2803A, U2 ULN2803A, U3 PCA9685PW

Commit message: Added Ordered JLC version
Parts:
- removed A3, A4, A5: A0, Jumper:SolderJumper-2_P1.3mm_Open_TrianglePad1.0x1.5mm
- U1, U2: footprint Package_SO:SOIC-18W_7.5x11.6mm_P1.27mm -> Package_DIP:DIP-18_W7.62mm
- moved J3 82.5 mm to (129.5, 62.7), turned to 0 degrees
- moved U2 76.6 mm to (117.0, 60.2), turned to 0 degrees
- moved C1 75.5 mm to (84.0, 57.5), turned to 180 degrees
- moved J1 73.6 mm to (98.0, 59.0), turned to 90 degrees
- moved J2 70.3 mm to (72.5, 80.5), turned to 180 degrees
- moved R9 66.6 mm to (100.5, 55.3)
- moved R8 66.6 mm to (103.7, 55.3)
- moved R7 60.9 mm to (111.0, 64.0), turned to 90 degrees
- moved R5 60.1 mm to (91.6, 64.9), turned to 90 degrees
- moved R6 58.3 mm to (99.1, 64.5), turned to 90 degrees
- moved C2 56.2 mm to (121.0, 83.2), turned to 0 degrees
- moved U1 56.2 mm to (87.5, 80.5), turned to 180 degrees
- moved R4 54.1 mm to (95.0, 64.9), turned to 90 degrees
- moved U3 54.1 mm to (102.9, 71.7)
- moved R1 37.0 mm to (98.0, 86.2)
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Connections:
- R1 pad 1: Net-(A3-A) -> Net-(A0-A)
- R2 pad 1: Net-(A2-A) -> Net-(A1-A)
- R3 pad 1: Net-(A1-A) -> Net-(A2-A)
- R4 pad 1: Net-(A0-A) -> Net-(U3-A3)
- U3 pad 1: Net-(A3-A) -> Net-(A0-A)
- U3 pad 2: Net-(A2-A) -> Net-(A1-A)
- U3 pad 3: Net-(A1-A) -> Net-(A2-A)
- U3 pad 4: Net-(A0-A) -> Net-(U3-A3)
Routing:
- net Net-(U3-A5): track 68.8 -> 13.2 mm
- net MCU_5V+: track 79.4 -> 133.4 mm
- net Net-(U3-A4): track 46.4 -> 10.6 mm
- net Net-(A3-A): track 35.0 -> 0.00 mm
- net MCU_3V3+: track 67.4 -> 42.5 mm, vias 7 -> 1
- net Net-(A0-A): track 15.2 -> 26.4 mm, vias 0 -> 2
- net /Signal7: track 4.97 -> 14.6 mm
- net MCU_SCL: track 25.5 -> 17.7 mm, vias 1 -> 0
- net Net-(U3-A3): track 0.00 -> 7.78 mm
- net /Signal6: track 6.51 -> 13.8 mm
- net MCU_SDA: track 24.4 -> 17.3 mm, vias 1 -> 0
- net /Signal8: track 5.04 -> 12.1 mm
- net MCU_GND: track 103.5 -> 97.0 mm, vias 0 -> 1
- net Net-(A1-A): track 20.3 -> 26.6 mm, vias 0 -> 2
- net /Signal5: track 8.05 -> 13.0 mm
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- added copper zone on B.Cu, net MCU_GND
Other:
- board size 47 x 34.5 mm -> 62 x 36 mm
- board text added: "16"
- board text added: "17"
- board text added: "CH0"
- board text added: "CH1"
- board text added: "CH2"
- board text added: "CH3"
- board text added: "CH4"
- board text added: "CH5"
- board text added: "CH6"
- board text added: "CH7"
- board text added: "V+"
- board text added: "VCC"
- board text removed: "0"
- board text removed: "1"
- board text removed: "10"
- board text removed: "11"
- board text removed: "2"
- board text removed: "3"
- board text removed: "3v3"
- board text removed: "4"
- board text removed: "5"
- board text removed: "5V"
- board text removed: "6"
- board text removed: "7"
- board text removed: "8"
- board text removed: "9"
- board text removed: "Ave's"
- board text removed: "I2C Haptic Module 16 Channel"
- board text removed: "JLCJLCJLCJLC"
- board text removed: "V0.1"
