File: PCB/Haptics PWM module/Haptics PWM module.kicad_sch (KiCad schematic)
At the start: 7 parts, among them J1 Conn_01x05_Pin, J2 JST_XH_FEMALE, J3 JST_XH_FEMALE_1, U1 ULN2803A, U2 ULN2803A

Commit message: Added Ordered JLC version
Parts:
- U1, U2: footprint Package_SO:SOIC-18W_7.5x11.6mm_P1.27mm -> Package_DIP:DIP-18_W7.62mm
Changed lines of the file:
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@@
 			)
 		)
-		(property "Footprint" "Package_SO:SOIC-18W_7.5x11.6mm_P1.27mm"
+		(property "Footprint" "Package_DIP:DIP-18_W7.62mm"
 			(at 215.9 138.43 0)
 			(effects
@@
 				)
 				(justify left)
-				(hide yes)
 			)
 		)
@@
 			)
 		)
-		(property "Footprint" "Package_SO:SOIC-18W_7.5x11.6mm_P1.27mm"
+		(property "Footprint" "Package_DIP:DIP-18_W7.62mm"
 			(at 215.9 80.01 0)
 			(effects
@@
 				)
 				(justify left)
-				(hide yes)
 			)
 		)
