File: PCB/Haptics PWM module/PCA_Module.kicad_sch (KiCad schematic)
At the start: 16 parts, among them U3 PCA9685PW

Commit message: Added Ordered JLC version
Parts:
- removed A0, A4, A5: A0, Jumper:SolderJumper-2_P1.3mm_Open_TrianglePad1.0x1.5mm, symbol Jumper:SolderJumper_2_Open
- renumbered A3 to A0, A2 to A1, A1 to A2
Other:
- note added: "Ground last three. No practical way to use more than 8 boards anyway"
- note added: "The traces should be cuttable"
